File: Nade.kicad_sch (KiCad schematic)
At the start: 44 parts, among them J1 FTSH-107-01-L-DV-K, J2 Conn_01x03_Pin, J3 UART_IN, J4 BATT, J5 MEM2085-00-115-00-A_REV0.2, J6 Conn_01x02_Pin, J8 Buzzer, Q1 NMOS, Q2 NMOS, SW2 SW_SPDT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

Commit message: v1
Parts:
- TP1, TP2, TP3: footprint TestPoint:TestPoint_Loop_D2.50mm_Drill1.85mm -> TestPoint:TestPoint_Pad_D1.5mm
- TP4: footprint TestPoint:TestPoint_Loop_D2.50mm_Drill1.85mm -> TestPoint:TestPoint_Pad_D1.0mm
Connections:
- net PA0: now also J5.CD; no longer U4.2 (GATE1)
- net PA2: no longer J5.CD
- net PB15: now also U4.5 (GATE2)
- net PB9: now also U4.2 (GATE1)
- net PC2: no longer U4.5 (GATE2)
Changed lines of the file:
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@@
 	(wire
 		(pts
+			(xy 46.99 62.23) (xy 57.15 62.23)
+		)
+		(stroke
+			(width 0)
+			(type default)
+		)
+	)
+	(wire
+		(pts
 			(xy 80.01 101.6) (xy 82.55 101.6)
 		)
@@
 	(wire
 		(pts
-			(xy 54.61 62.23) (xy 57.15 62.23)
-		)
-		(stroke
-			(width 0)
-			(type default)
-		)
-	)
-	(wire
-		(pts
 			(xy 156.21 114.3) (xy 156.21 123.19)
 		)
@@
 		)
 	)
-	(label "PA0"
+	(label "PB9"
 		(at 28.575 171.45 0)
 		(effects
@@
 		)
 	)
-	(label "PA2"
+	(label "PA12"
+		(at 46.99 62.23 0)
+		(effects
+			(font
+				(size 1.27 1.27)
+			)
+			(justify left bottom)
+		)
+	)
+	(label "PA0"
 		(at 353.695 39.37 0)
 		(effects
@@
 		)
 	)
-	(label "PC2"
+	(label "PB15"
 		(at 88.9 171.45 0)
 		(effects
@@
 		)
 	)
-	(global_label "PA12"
-		(shape input)
-		(at 54.61 62.23 180)
-		(fields_autoplaced yes)
-		(effects
-			(font
-				(size 1.27 1.27)
-			)
-			(justify right)
-		)
-		(property "Intersheetrefs" "${INTERSHEET_REFS}"
-			(at 46.8472 62.23 0)
-			(effects
-				(font
-					(size 1.27 1.27)
-				)
-				(justify right)
-				(hide yes)
-			)
-		)
-	)
 	(global_label "VDD"
 		(shape output)
@@
 		(length 2.54)
 		(shape round)
+		(at 186.69 151.13 0)
+		(fields_autoplaced yes)
+		(effects
+			(font
+				(size 1.27 1.27)
+			)
+			(justify left bottom)
+		)
+		(property "Netclass" "VDD"
+			(at 187.3885 148.59 0)
+			(effects
+				(font
+					(size 1.27 1.27)
+				)
+				(justify left)
+			)
+		)
+		(property "Component Class" ""
+			(at -30.48 97.79 0)
+			(effects
+				(font
+					(size 1.27 1.27)
+					(italic yes)
+				)
+			)
+		)
+	)
+	(netclass_flag ""
+		(length 2.54)
+		(shape round)
+		(at 214.63 123.19 0)
+		(fields_autoplaced yes)
+		(effects
+			(font
+				(size 1.27 1.27)
+			)
+			(justify left bottom)
+		)
+		(property "Netclass" "VDD"
+			(at 215.3285 120.65 0)
+			(effects
+				(font
+					(size 1.27 1.27)
+				)
+				(justify left)
+			)
+		)
+		(property "Component Class" ""
+			(at -2.54 69.85 0)
+			(effects
+				(font
+					(size 1.27 1.27)
+					(italic yes)
+				)
+			)
+		)
+	)
+	(netclass_flag ""
+		(length 2.54)
+		(shape round)
+		(at 171.45 151.13 0)
+		(fields_autoplaced yes)
+		(effects
+			(font
+				(size 1.27 1.27)
+			)
+			(justify left bottom)
+		)
+		(property "Netclass" "VDD"
+			(at 172.1485 148.59 0)
+			(effects
+				(font
+					(size 1.27 1.27)
+				)
+				(justify left)
+			)
+		)
+		(property "Component Class" ""
+			(at -45.72 97.79 0)
+			(effects
+				(font
+					(size 1.27 1.27)
+					(italic yes)
+				)
+			)
+		)
+	)
+	(netclass_flag ""
+		(length 2.54)
+		(shape round)
+		(at 143.51 115.57 0)
+		(effects
+			(font
+				(size 1.27 1.27)
+			)
+			(justify left bottom)
+		)
+		(property "Netclass" "VDD"
+			(at 142.9385 111.125 0)
+			(effects
+				(font
+					(size 1.27 1.27)
+				)
+				(justify left)
+			)
+		)
+		(property "Component Class" ""
+			(at -73.66 62.23 0)
+			(effects
+				(font
+					(size 1.27 1.27)
+					(italic yes)
+				)
+			)
+		)
+	)
+	(netclass_flag ""
+		(length 2.54)
+		(shape round)
 		(at 147.32 39.37 0)
 		(fields_autoplaced yes)
@@
 		)
 	)
+	(netclass_flag ""
+		(length 2.54)
+		(shape round)
+		(at 149.86 99.06 0)
+		(fields_autoplaced yes)
+		(effects
+			(font
+				(size 1.27 1.27)
+			)
+			(justify left bottom)
+		)
+		(property "Netclass" "VDD"
+			(at 150.5585 96.52 0)
+			(effects
+				(font
+					(size 1.27 1.27)
+				)
+				(justify left)
+			)
+		)
+		(property "Component Class" ""
+			(at -67.31 45.72 0)
+			(effects
+				(font
+					(size 1.27 1.27)
+					(italic yes)
+				)
+			)
+		)
+	)
+	(netclass_flag ""
+		(length 2.54)
+		(shape round)
+		(at 187.96 109.22 180)
+		(fields_autoplaced yes)
+		(effects
+			(font
+				(size 1.27 1.27)
+			)
+			(justify right bottom)
+		)
+		(property "Netclass" "VDD"
+			(at 188.6585 111.76 0)
+			(effects
+				(font
+					(size 1.27 1.27)
+				)
+				(justify left)
+			)
+		)
+		(property "Component Class" ""
+			(at -29.21 55.88 0)
+			(effects
+				(font
+					(size 1.27 1.27)
+					(italic yes)
+				)
+			)
+		)
+	)
 	(symbol
 		(lib_id "Grenade:INA213AIRSWR")
@@
 			)
 		)
-		(property "Footprint" "TestPoint:TestPoint_Loop_D2.50mm_Drill1.85mm"
+		(property "Footprint" "TestPoint:TestPoint_Pad_D1.5mm"
 			(at 228.6 86.36 0)
 			(effects
@@
 			)
 		)
-		(property "Footprint" "TestPoint:TestPoint_Loop_D2.50mm_Drill1.85mm"
+		(property "Footprint" "TestPoint:TestPoint_Pad_D1.0mm"
 			(at 204.47 109.22 0)
 			(effects
@@
 			)
 		)
-		(property "Footprint" "TestPoint:TestPoint_Loop_D2.50mm_Drill1.85mm"
+		(property "Footprint" "TestPoint:TestPoint_Pad_D1.5mm"
 			(at 220.98 91.44 0)
 			(effects
@@
 			)
 		)
-		(property "Footprint" "TestPoint:TestPoint_Loop_D2.50mm_Drill1.85mm"
+		(property "Footprint" "TestPoint:TestPoint_Pad_D1.5mm"
 			(at 154.94 105.41 0)
 			(effects

Commit message: v2
Parts:
- removed J3: UART_IN, Connector_JST:JST_SH_BM02B-SRSS-TB_1x02-1MP_P1.00mm_Vertical, symbol Connector:Conn_01x02_Pin
- added J3: Extra, Connector_PinHeader_1.27mm:PinHeader_2x07_P1.27mm_Vertical_SMD, symbol Connector:Conn_01x14_Pin
- added J7: UART, Connector_JST:JST_SH_SM04B-SRSS-TB_1x04-1MP_P1.00mm_Horizontal, symbol Connector:Conn_01x04_Pin
- TP5: footprint TestPoint:TestPoint_Loop_D2.50mm_Drill1.85mm -> TestPoint:TestPoint_THTPad_2.0x2.0mm_Drill1.0mm
Connections:
- net GND: now also J7.4 (Pin_4)
- net VDD: now also J7.3 (Pin_3)
- net at MCU1.10 (PB12): now also J3.5 (Pin_5)
- net at MCU1.11 (PB13): now also J3.6 (Pin_6)
- net at MCU1.29 (PB6): now also J7.1 (Pin_1)
- net at MCU1.30 (PB7): now also J7.2 (Pin_2)
- net at MCU1.35 (PC6): now also J3.14 (Pin_14)
- net at MCU1.6 (PA9): now also J3.1 (Pin_1)
- net at MCU1.7 (PC13): now also J3.2 (Pin_2)
- net at MCU1.8 (PB11): now also J3.3 (Pin_3)
- net at MCU1.9 (PB10): now also J3.4 (Pin_4)
- net PA12: no longer names the net of MCU1.18 (PA12)
- net PA12: now also J3.7 (Pin_7)
- net PA5: no longer names the net of MCU1.50 (PA5)
- net PA5: now also J3.10 (Pin_10)
- net PA8: no longer names the net of MCU1.49 (PA8)
- net PA8: now also J3.11 (Pin_11)
- net PB14: no longer names the net of MCU1.19 (PB14)
- net PB14: now also J3.8 (Pin_8)
- net PB8: no longer names the net of MCU1.40 (PB8)
- net PB8: now also J3.13 (Pin_13)
- net PC2: no longer names the net of MCU1.48 (PC2)
- net PC2: now also J3.12 (Pin_12)
- new net: J3.9 (Pin_9), MCU1.27 (PB5)
Other:
- moved on the sheet: D1, D2, SW3, U4
