File: Nade.kicad_pcb (KiCad board)
At the start: 4 copper layers, 30 x 30 mm, 44 parts, among them J1 FTSH-107-01-L-DV-K, J2 Conn_01x03_Pin, J3 UART_IN, J4 BATT, J5 MEM2085-00-115-00-A_REV0.2, J6 Conn_01x02_Pin, J8 Buzzer, Q1 NMOS, Q2 NMOS, SW2 SW_SPDT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

Commit message: v1
Parts:
- J3, Q1, R16, R17: moved to B.Cu
- J5, R14, SW3: moved to F.Cu
- TP1: footprint TestPoint:TestPoint_Loop_D2.50mm_Drill1.85mm -> TestPoint:TestPoint_Pad_D1.5mm; moved to B.Cu
- TP2, TP3: footprint TestPoint:TestPoint_Loop_D2.50mm_Drill1.85mm -> TestPoint:TestPoint_Pad_D1.5mm
- TP4: footprint TestPoint:TestPoint_Loop_D2.50mm_Drill1.85mm -> TestPoint:TestPoint_Pad_D1.0mm
- moved TP1 62.0 mm to (120.3, 87.8), turned to 180 degrees
- moved TP4 60.2 mm to (125.9, 84.3)
- moved TP3 43.9 mm to (139.7, 89.1)
- moved TP2 42.6 mm to (139.7, 92.9)
- moved TP5 42.2 mm to (143.3, 94.7)
- moved J5 23.4 mm to (126.7, 91.5), turned to 90 degrees
- moved J4 21.3 mm to (118.6, 101.3), turned to -90 degrees
- moved J3 20.3 mm to (138.7, 108.0)
- moved J8 20.1 mm to (117.2, 108.7)
- moved R8 19.7 mm to (116.6, 91.6), turned to 180 degrees
- moved D1 18.0 mm to (143.3, 98.9)
- moved R9 16.2 mm to (115.0, 98.1), turned to 90 degrees
- moved D2 15.9 mm to (145.8, 98.9), turned to 180 degrees
- moved R16 15.7 mm to (133.0, 103.4), turned to 0 degrees
- moved SW3 15.5 mm to (118.2, 102.4), turned to 90 degrees
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Connections:
- net PA12 renamed /PA12
- J5 pad CD: /PA2 -> /PA0
- U4 pad 2: /PA0 -> /PB9
- U4 pad 5: /PC2 -> /PB15
Routing:
- net GND: track 10.9 -> 104.9 mm, vias 6 -> 76
- net VDD: track 3.19 -> 55.5 mm, vias 5 -> 31
- net /PA11: track 0.89 -> 37.2 mm, vias 0 -> 3
- net RESET': track 0.00 -> 30.1 mm, vias 0 -> 4
- net /PB2: track 0.00 -> 27.4 mm, vias 0 -> 2
- net /PA4: track 0.00 -> 21.0 mm, vias 0 -> 3
- net Net-(U1-OUT): track 6.10 -> 25.0 mm, vias 0 -> 1
- net /PA6: track 0.00 -> 18.2 mm, vias 0 -> 2
- net Net-(J2-Pin_2): track 0.00 -> 13.3 mm, vias 0 -> 1
- net /PA7: track 0.00 -> 12.8 mm, vias 0 -> 2
- net Net-(J8-Pin_2): track 0.00 -> 11.7 mm
- net /PA15: track 0.00 -> 10.5 mm, vias 0 -> 1
- net Net-(J6-Pin_2): track 0.00 -> 10.4 mm, vias 0 -> 1
- net /PA1: track 0.00 -> 10.3 mm, vias 0 -> 2
- net /PA2: track 0.00 -> 10.1 mm, vias 0 -> 1
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Other:
- board size 30 x 30 mm -> 35 x 35 mm

Commit message: v2
Parts:
- removed TP5: GND, TestPoint:TestPoint_Loop_D2.50mm_Drill1.85mm
- added GND: GND, TestPoint:TestPoint_THTPad_2.0x2.0mm_Drill1.0mm, F.Cu at (144.6, 95.8)
- added UART: UART, Connector_JST:JST_SH_SM04B-SRSS-TB_1x04-1MP_P1.00mm_Horizontal, B.Cu at (138.2, 109.1)
- J3: value UART_IN -> Extra; footprint Connector_JST:JST_SH_BM02B-SRSS-TB_1x02-1MP_P1.00mm_Vertical -> Connector_PinHeader_1.27mm:PinHeader_2x07_P1.27mm_Vertical_SMD
- moved J3 15.3 mm to (138.0, 92.7), turned to -90 degrees
- moved C10 2.51 mm to (133.7, 85.7)
- moved C6 2.51 mm to (135.0, 86.4)
- moved C5 2.51 mm to (135.2, 85.4)
- renumbered J8 to Buzz, J6 to Pyro, TP3 to VDD1, TP2 to VDD2
Connections:
- MCU1 pad 10: unconnected-(MCU1-PB12-Pad10) -> Net-(J3-Pin_5)
- MCU1 pad 11: unconnected-(MCU1-PB13-Pad11) -> Net-(J3-Pin_6)
- MCU1 pad 18: /PA12 -> Net-(J3-Pin_7)
- MCU1 pad 19: /PB14 -> Net-(J3-Pin_8)
- MCU1 pad 29: Net-(J3-Pin_1) -> Net-(J7-Pin_1)
- MCU1 pad 30: Net-(J3-Pin_2) -> Net-(J7-Pin_2)
- MCU1 pad 35: unconnected-(MCU1-PC6-Pad35) -> Net-(J3-Pin_14)
- MCU1 pad 40: /PB8 -> Net-(J3-Pin_13)
- MCU1 pad 48: /PC2 -> Net-(J3-Pin_12)
- MCU1 pad 49: /PA8 -> Net-(J3-Pin_11)
- MCU1 pad 50: /PA5 -> Net-(J3-Pin_10)
- MCU1 pad 6: unconnected-(MCU1-PA9-Pad6) -> Net-(J3-Pin_1)
- MCU1 pad 7: unconnected-(MCU1-PC13-Pad7) -> Net-(J3-Pin_2)
- MCU1 pad 8: unconnected-(MCU1-PB11-Pad8) -> Net-(J3-Pin_3)
- MCU1 pad 9: unconnected-(MCU1-PB10-Pad9) -> Net-(J3-Pin_4)
Routing:
- net Net-(J3-Pin_11): track 0.00 -> 37.3 mm, vias 0 -> 2
- net Net-(J3-Pin_7): track 0.00 -> 35.5 mm, vias 0 -> 3
- net Net-(J3-Pin_8): track 0.00 -> 33.9 mm, vias 0 -> 3
- net Net-(J3-Pin_5): track 0.00 -> 29.6 mm, vias 0 -> 2
- net Net-(J3-Pin_6): track 0.00 -> 28.3 mm, vias 0 -> 3
- net Net-(J3-Pin_3): track 0.00 -> 27.7 mm, vias 0 -> 2
- net Net-(J3-Pin_4): track 0.00 -> 25.8 mm, vias 0 -> 3
- net Net-(J3-Pin_10): track 0.00 -> 23.7 mm, vias 0 -> 2
- net Net-(J3-Pin_1): track 4.14 -> 22.3 mm
- net Net-(J3-Pin_12): track 0.00 -> 16.7 mm, vias 0 -> 1
- net Net-(J3-Pin_2): track 4.20 -> 19.9 mm, vias 1 -> 2
- net Net-(J3-Pin_14): track 0.00 -> 13.5 mm, vias 0 -> 2
- net GND: track 104.9 -> 117.7 mm, vias 76 -> 78
- net Net-(J3-Pin_13): track 0.00 -> 12.1 mm, vias 0 -> 1
- net VDD: track 55.5 -> 59.3 mm
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Other:
- board text added: "+"
- board text added: "-"
- board text added: "10"
- board text added: "11"
- board text added: "18"
- board text added: "19"
- board text added: "27"
- board text added: "29"
- board text added: "30"
- board text added: "35"
- board text added: "40"
- board text added: "48"
- board text added: "49"
- board text added: "50"
- board text added: "6"
- board text added: "7"
- board text added: "8"
- board text added: "9"
- board text added: "VRAW"

Commit message: v5
Parts:
- removed the GND at (144.6, 95.8)
- removed J5: MEM2085-00-115-00-A_REV0.2, footprints:GCT_MEM2085-00-115-00-A_REV0.2
- removed UART: UART, Connector_JST:JST_SH_SM04B-SRSS-TB_1x04-1MP_P1.00mm_Horizontal
- removed VDD1, VDD2: VDD, TestPoint:TestPoint_Pad_D1.5mm
- added GND: GND, TestPoint:TestPoint_THTPad_D1.5mm_Drill0.7mm, F.Cu at (140.2, 109.0)
- added IC1: MB85RS2MTYPNF-G-AWERE2, footprints:SOIC127P600X175-8N, B.Cu at (125.1, 99.0)
- added J7: UART, Connector_JST:JST_SH_SM04B-SRSS-TB_1x04-1MP_P1.00mm_Horizontal, B.Cu at (138.9, 104.3)
- added VDD: VDD, TestPoint:TestPoint_Pad_D1.5mm, F.Cu at (139.9, 101.1)
- added VDD: VDD, TestPoint:TestPoint_Pad_D1.5mm, B.Cu at (130.6, 92.2)
- Buzz, R14: moved to B.Cu
- C10, C5, C6, C7, C8, C9, L1, R10, R11, R12, U1, U2: moved to F.Cu
- R8, R9: value 47 -> 10k
- TP4: footprint TestPoint:TestPoint_Pad_D1.0mm -> TestPoint:TestPoint_Pad_D1.5mm
- U3: value ADXL314WBCPZ-RL -> ADXL373BCCZ-RL7; footprint footprints:LFCSP32_CP-32-17_ADI -> footprints:ADXL373
- moved TP1 14.2 mm to (134.5, 88.9)
- moved L1 12.9 mm to (137.5, 92.6), turned to -90 degrees
- moved SW2 12.6 mm to (132.5, 87.7), turned to -90 degrees
- moved R14 11.3 mm to (130.4, 95.8), turned to 0 degrees
- moved R15 11.2 mm to (126.7, 103.2), turned to 0 degrees
- moved J4 11.1 mm to (124.9, 92.2), turned to 0 degrees
- moved U1 10.9 mm to (135.2, 91.2)
- moved D1 9.66 mm to (139.3, 90.1), turned to -150 degrees
- moved D2 8.85 mm to (140.1, 92.2), turned to -150 degrees
- moved U4 8.25 mm to (141.7, 95.2), turned to -60 degrees
- moved C7 8.02 mm to (133.4, 91.6)
- moved R18 6.22 mm to (142.8, 103.3)
- moved C9 6.20 mm to (134.3, 93.4)
- moved TP4 6.17 mm to (121.9, 89.0)
- moved R9 5.54 mm to (120.3, 96.5), turned to 180 degrees
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Connections:
- C8 pad 1: Net-(U1-OUT) -> VDD
- C9 pad 1: Net-(U1-OUT) -> VDD
- MCU1 pad 27: /PB5 -> Net-(J3-Pin_9)
- MCU1 pad 28: (no net) -> /PB5
- R10 pad 1: VDD -> Net-(R10-Pad1)
- R10 pad 2: Net-(U1-OUT) -> VDD
- R13 pad 1: /PA7 -> /PA4
- R14 pad 1: /PA4 -> /PA6
- R15 pad 1: /PA6 -> /PA7
- U1 pad D3: Net-(U1-OUT) -> VDD
- U2 pad 2: Net-(U1-OUT) -> VDD
- U2 pad 3: Net-(U1-OUT) -> VDD
- U2 pad 4: VDD -> Net-(R10-Pad1)
- U2 pad 5: VDD -> Net-(R10-Pad1)
- U3 pad 1: GND -> VDD
- U3 pad 12: unconnected-(U3-NC-Pad12) -> GND
- U3 pad 13: unconnected-(U3-NC-Pad13) -> GND
- U3 pad 14: unconnected-(U3-NC-Pad14) -> VDD
- U3 pad 16: unconnected-(U3-NC-Pad16) -> GND
- U3 pad 3: GND -> unconnected-(U3-RESERVED-Pad3)
- U3 pad 5: VDD -> unconnected-(U3-RESERVED-Pad5)
- U3 pad 6: VDD -> /PC1
- U3 pad 7: unconnected-(U3-RESERVED-Pad7) -> VDD
- U3 pad 8: unconnected-(U3-NC-Pad8) -> /PC0
Routing:
- net GND: track 117.7 -> 51.2 mm, vias 78 -> 47
- net Net-(J3-Pin_11): track 37.3 -> 9.67 mm, vias 2 -> 1
- net Net-(U1-OUT): track 25.0 -> 0.00 mm, vias 1 -> 0
- net Net-(J3-Pin_9): track 0.00 -> 19.0 mm, vias 0 -> 2
- net /PA4: track 24.2 -> 7.80 mm, vias 3 -> 1
- net Net-(J3-Pin_7): track 35.5 -> 23.5 mm, vias 3 -> 2
- net VDD: track 59.3 -> 49.3 mm
- net Net-(J3-Pin_5): track 29.6 -> 19.6 mm
- net /PA6: track 18.2 -> 8.53 mm, vias 2 -> 1
- net Net-(J3-Pin_3): track 27.7 -> 18.3 mm
- net Net-(J3-Pin_1): track 22.3 -> 14.3 mm, vias 1 -> 2
- net Net-(J3-Pin_8): track 33.9 -> 26.5 mm, vias 3 -> 2
- net Net-(R10-Pad1): track 0.00 -> 6.86 mm, vias 0 -> 1
- net Net-(J8-Pin_2): track 11.7 -> 4.90 mm
- net Net-(J3-Pin_10): track 23.7 -> 17.3 mm
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- added copper zone on In1.Cu, net GND
- added copper zone on In2.Cu, net VDD
- removed copper zone on In2.Cu, net GND
- removed copper zone on In1.Cu, net VDD
Other:
- board size 35 x 35 mm -> 30 x 30 mm
- board text added: "VDIV"
- board text added: "x"
- board text removed: "29"
- board text removed: "30"
- board text removed: "VRAW"
