File: _autosave-Nade.kicad_sch (KiCad schematic)
At the start: 45 parts, among them IC1 MB85RS2MTYPNF-G-AWERE2, J1 FTSH-107-01-L-DV-K, J2 Conn_01x03_Pin, J3 Extra, J4 BATT, J6 Conn_01x02_Pin, J7 UART, J8 Buzzer, Q1 NMOS, Q2 NMOS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

Commit message: v5
Parts:
- IC1: footprint SOIC127P600X175-8N -> footprints:SOIC127P600X175-8N
- TP4: footprint TestPoint:TestPoint_Pad_D1.0mm -> TestPoint:TestPoint_Pad_D1.5mm
- TP5: footprint TestPoint:TestPoint_THTPad_2.0x2.0mm_Drill1.0mm -> TestPoint:TestPoint_THTPad_D1.5mm_Drill0.7mm
Changed lines of the file:
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@@
 			)
 		)
-		(property "Footprint" "SOIC127P600X175-8N"
+		(property "Footprint" "footprints:SOIC127P600X175-8N"
 			(at 319.405 134.29 0)
 			(effects
@@
 			)
 		)
-		(property "Footprint" "TestPoint:TestPoint_THTPad_2.0x2.0mm_Drill1.0mm"
+		(property "Footprint" "TestPoint:TestPoint_THTPad_D1.5mm_Drill0.7mm"
 			(at 156.21 143.51 0)
 			(effects
@@
 			)
 		)
-		(property "Footprint" "TestPoint:TestPoint_Pad_D1.0mm"
+		(property "Footprint" "TestPoint:TestPoint_Pad_D1.5mm"
 			(at 204.47 109.22 0)
 			(effects
